File: kicad/sram.kicad_sch (KiCad schematic)
At the start: 7 parts, among them U13 74LS139, U19 74HC86, U2 IS61C1024-15N, U3 IS61C1024-15N, U4 IS61C1024-15N, U5 IS61C1024-15N

Commit message: add description for JP1
Other:
- note added: "JP1 1-2 pin 30 is Vcc 28-pin DIP 32-pin DIP ≤ 2 Mbit 2-3 pin 30 is A19 32-pin DIP > 2 Mbit"
Changed lines of the file:
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@@
+		)
+	)
+	(text "JP1\n1-2	pin 30 is Vcc\n	28-pin DIP\n	32-pin DIP ≤ 2 Mbit\n2-3	pin 30 is A19\n	32-pin DIP > 2 Mbit"
+		(exclude_from_sim no)
+		(at 116.586 55.118 0)
+		(effects
+			(font
+				(face "KiCad Font")
+				(size 1.27 1.27)
+			)
+			(justify left)
 		)
 	)
